File: dc-dc-buck-stm8/buck-stm8.sch (KiCad schematic (older format))
At the start: 37 parts

Commit message: pcb voltage-dc-dc-buck-stm8
Parts:
- removed Q?: Q_NMOS_DGS, symbol Q_NMOS_DGS
- removed U?: LM7805, symbol LM7805
- added C11: 100nF, Capacitors_SMD:C_0805_HandSoldering, symbol C
- added Q2: Q_PMOS_GSD, TO_SOT_Packages_THT:TO-220_Neutral123_Vertical, symbol Q_PMOS_GSD
- added R12: R, Resistors_ThroughHole:Resistor_Horizontal_RM10mm, symbol R
- added U1: LM7805CT, TO_SOT_Packages_SMD:TO-252-2Lead, symbol LM7805CT
- C1, C10, C3, C4, C6, C8, C9: renamed from C?; footprint (none) -> Capacitors_SMD:C_0805_HandSoldering
- C2, C5: renamed from C?; footprint (none) -> Capacitors_SMD:c_elec_8x10.5
- C7: renamed from C?; footprint (none) -> Capacitors_SMD:C_1206_HandSoldering
- D1, D3: renamed from D?; footprint (none) -> Diodes_SMD:SOD-123
- D2: renamed from D?; footprint (none) -> Diodes_SMD:DO-214AB
- D4: renamed from D?; footprint (none) -> Diodes_SMD:DO-214AB_Handsoldering
- D5: renamed from D?; footprint (none) -> LEDs:LED_0805
- F1: renamed from F?; footprint (none) -> Fuse_Holders_and_Fuses:Fuseholder5x20_horiz_open_lateral_Type-II
- IC1: renamed from IC?; footprint TSSOP-20 -> Housings_SSOP:TSSOP-20_4.4x6.5mm_Pitch0.65mm
- L1: renamed from L?; footprint (none) -> Inductors:SELF-WE-PD-XXL
- P1, P2: renamed from P?; footprint (none) -> Terminal_Blocks:TerminalBlock_Pheonix_PT-3.5mm_2pol
- P3: renamed from P?; footprint (none) -> Pin_Headers:Pin_Header_Straight_1x04
- Q1, Q4: renamed from Q?; footprint TO-220 -> TO_SOT_Packages_SMD:SOT-23
- Q3: renamed from Q?; footprint (none) -> TO_SOT_Packages_SMD:SOT-23
- R1, R10, R11, R2, R3, R4, R5, R6, R7, R8: renamed from R?; footprint (none) -> Resistors_SMD:R_0805_HandSoldering
- R9: renamed from R?; footprint (none) -> Resistors_ThroughHole:Resistor_Horizontal_RM10mm
Connections:
- wire segments 81 -> 86
