File: ctrl-power-peltier/ctrl-power-peltier.sch (KiCad schematic (older format))
At the start: 39 parts, among them IC1 STM8S003F3P, P1 CONN_01X02, P2 CONN_01X02, P3 CONN_01X04, Q1 2SC1815, Q2 Q_PMOS_GSD, Q3 2SA1015, Q4 2SC1815, U1 LM7805CT

Commit message: pcb voltage-dc-dc-buck-stm8
Parts:
- removed C11: 100nF, Capacitors_SMD:C_0805_HandSoldering, symbol C
- removed Q2: Q_PMOS_GSD, TO_SOT_Packages_THT:TO-220_Neutral123_Vertical, symbol Q_PMOS_GSD
- removed R12: R, Resistors_ThroughHole:Resistor_Horizontal_RM10mm, symbol R
- removed U1: LM7805CT, TO_SOT_Packages_SMD:TO-252-2Lead, symbol LM7805CT
- added Q?: Q_NMOS_DGS, symbol Q_NMOS_DGS
- added U?: LM7805, TO_SOT_Packages_SMD:TO-252-2Lead, symbol LM7805
- C?: renamed from C5; footprint Capacitors_SMD:c_elec_8x10.5 -> (none)
- C?: renamed from C2; footprint Capacitors_SMD:c_elec_8x10.5 -> (none)
- C?: renamed from C6; footprint Capacitors_SMD:C_0805_HandSoldering -> (none)
- C?: renamed from C7; footprint Capacitors_SMD:C_1206_HandSoldering -> Capacitors_SMD:C_0805_HandSoldering
- D?: renamed from D1; footprint Diodes_SMD:SOD-123 -> (none)
- D?: renamed from D3; footprint Diodes_SMD:SOD-123 -> (none)
- D?: renamed from D4; footprint Diodes_SMD:DO-214AB_Handsoldering -> (none)
- D?: renamed from D2; footprint Diodes_SMD:DO-214AB -> (none)
- D?: renamed from D5; footprint LEDs:LED_0805 -> (none)
- F?: renamed from F1; footprint Fuse_Holders_and_Fuses:Fuseholder5x20_horiz_open_lateral_Type-II -> (none)
- IC?: renamed from IC1; footprint Housings_SSOP:TSSOP-20_4.4x6.5mm_Pitch0.65mm -> TSSOP-20
- L?: renamed from L1; footprint Inductors:SELF-WE-PD-XXL -> (none)
- P?: renamed from P1; footprint Terminal_Blocks:TerminalBlock_Pheonix_PT-3.5mm_2pol -> (none)
- P?: renamed from P3; footprint Pin_Headers:Pin_Header_Straight_1x04 -> (none)
- P?: renamed from P2; footprint Terminal_Blocks:TerminalBlock_Pheonix_PT-3.5mm_2pol -> (none)
- Q?: renamed from Q1; footprint TO_SOT_Packages_SMD:SOT-23 -> TO_SOT_Packages_SMD:SOT-23_Handsoldering
- Q?: renamed from Q3; footprint TO_SOT_Packages_SMD:SOT-23 -> TO_SOT_Packages_SMD:SOT-23_Handsoldering
- Q?: renamed from Q4; footprint TO_SOT_Packages_SMD:SOT-23 -> TO_SOT_Packages_SMD:SOT-23_Handsoldering
- R?: renamed from R5; footprint Resistors_SMD:R_0805_HandSoldering -> (none)
- R?: renamed from R8; footprint Resistors_SMD:R_0805_HandSoldering -> (none)
- R?: renamed from R11; footprint Resistors_SMD:R_0805_HandSoldering -> (none)
- R?: renamed from R9; footprint Resistors_ThroughHole:Resistor_Horizontal_RM10mm -> (none)
- renumbered C4 to C?, C1 to C?, C3 to C?, C9 to C?, C10 to C?, C8 to C?, R4 to R?, R1 to R?, R6 to R?, R2 to R?, R3 to R?, R7 to R?, R10 to R?
Connections:
- wire segments 86 -> 81

Commit message: add pcb current-source
Parts:
- removed Q?: Q_NMOS_DGS, symbol Q_NMOS_DGS
- added F?: FUSE, symbol FUSE
- added Q?: Q_PMOS_GSD, TO_SOT_Packages_THT:TO-220_Neutral123_Vertical, symbol Q_PMOS_GSD
- added R? (x2): R, symbol R
- added U?: LM358, symbol LM358
Connections:
- net labels added: v_i
- wire segments 81 -> 90
Other:
- moved on the sheet: C?, P?, R?, U?
Changed lines of the file:
@@
-$EndComp
-$Comp
-L Q_NMOS_DGS Q?
-U 1 1 57D2DA53
-P 6700 1700
-F 0 "Q?" H 7000 1750 50  0000 R CNN
-F 1 "Q_NMOS_DGS" H 7350 1650 50  0000 R CNN
-F 2 "" H 6900 1800 50  0000 C CNN
-F 3 "" H 6700 1700 50  0000 C CNN
-	1    6700 1700
-	1    0    0    -1
 $EndComp
 $Comp
@@
 L R R?
 U 1 1 57D47909
-P 7100 4700
-F 0 "R?" V 7180 4700 50  0000 C CNN
-F 1 "R" V 7100 4700 50  0000 C CNN
-F 2 "" V 7030 4700 50  0000 C CNN
-F 3 "" H 7100 4700 50  0000 C CNN
-	1    7100 4700
+P 5750 4450
+F 0 "R?" V 5830 4450 50  0000 C CNN
+F 1 "R" V 5750 4450 50  0000 C CNN
+F 2 "" V 5680 4450 50  0000 C CNN
+F 3 "" H 5750 4450 50  0000 C CNN
+	1    5750 4450
 	0    1    1    0
 $EndComp
@@
 L CONN_01X02 P?
 U 1 1 57D47F46
-P 10450 1450
-F 0 "P?" H 10450 1600 50  0000 C CNN
-F 1 "CONN_01X02" V 10550 1450 50  0000 C CNN
-F 2 "" H 10450 1450 50  0000 C CNN
-F 3 "" H 10450 1450 50  0000 C CNN
-	1    10450 1450
-	1    0    0    -1
-$EndComp
-Text GLabel 9900 1400 0    60   Input ~ 0
+P 10850 900
+F 0 "P?" H 10850 1050 50  0000 C CNN
+F 1 "CONN_01X02" V 10950 900 50  0000 C CNN
+F 2 "" H 10850 900 50  0000 C CNN
+F 3 "" H 10850 900 50  0000 C CNN
+	1    10850 900
+	1    0    0    -1
+$EndComp
+Text GLabel 10300 850  0    60   Input ~ 0
 Vout
 Wire Wire Line
-	9900 1400 10250 1400
+	10300 850  10650 850
 $Comp
 L GND #PWR?
 U 1 1 57D48D36
-P 10100 1650
-F 0 "#PWR?" H 10100 1400 50  0001 C CNN
-F 1 "GND" H 10100 1500 50  0000 C CNN
-F 2 "" H 10100 1650 50  0000 C CNN
-F 3 "" H 10100 1650 50  0000 C CNN
-	1    10100 1650
-	1    0    0    -1
-$EndComp
-Wire Wire Line
-	10250 1500 10100 1500
-Wire Wire Line
-	10100 1500 10100 1650
+P 10500 2650
+F 0 "#PWR?" H 10500 2400 50  0001 C CNN
+F 1 "GND" H 10500 2500 50  0000 C CNN
+F 2 "" H 10500 2650 50  0000 C CNN
+F 3 "" H 10500 2650 50  0000 C CNN
+	1    10500 2650
+	1    0    0    -1
+$EndComp
+Wire Wire Line
+	10650 950  10500 950
 $Comp
 L LM7805 U?
 U 1 1 57D49FEF
-P 8000 4750
-F 0 "U?" H 8150 4554 50  0000 C CNN
-F 1 "LM7805" H 8000 4950 50  0000 C CNN
-F 2 "TO_SOT_Packages_SMD:TO-252-2Lead" V 8000 4750 50  0001 C CNN
-F 3 "" H 8000 4750 50  0000 C CNN
-	1    8000 4750
+P 6650 4500
+F 0 "U?" H 6800 4304 50  0000 C CNN
+F 1 "LM7805" H 6650 4700 50  0000 C CNN
+F 2 "TO_SOT_Packages_SMD:TO-252-2Lead" V 6650 4500 50  0001 C CNN
+F 3 "" H 6650 4500 50  0000 C CNN
+	1    6650 4500
 	1    0    0    -1
 $EndComp
@@
 L GND #PWR?
 U 1 1 57D4A727
-P 8000 5250
-F 0 "#PWR?" H 8000 5000 50  0001 C CNN
-F 1 "GND" H 8000 5100 50  0000 C CNN
-F 2 "" H 8000 5250 50  0000 C CNN
-F 3 "" H 8000 5250 50  0000 C CNN
-	1    8000 5250
-	1    0    0    -1
-$EndComp
-Wire Wire Line
-	8000 5000 8000 5250
-Wire Wire Line
-	7250 4700 7600 4700
+P 6650 5000
+F 0 "#PWR?" H 6650 4750 50  0001 C CNN
+F 1 "GND" H 6650 4850 50  0000 C CNN
+F 2 "" H 6650 5000 50  0000 C CNN
+F 3 "" H 6650 5000 50  0000 C CNN
+	1    6650 5000
+	1    0    0    -1
+$EndComp
+Wire Wire Line
+	6650 4750 6650 5000
+Wire Wire Line
+	5900 4450 6250 4450
 $Comp
 L +5V #PWR?
 U 1 1 57D4A9D6
-P 8800 4550
-F 0 "#PWR?" H 8800 4400 50  0001 C CNN
-F 1 "+5V" H 8800 4690 50  0000 C CNN
-F 2 "" H 8800 4550 50  0000 C CNN
-F 3 "" H 8800 4550 50  0000 C CNN
-	1    8800 4550
+P 7450 4300
+F 0 "#PWR?" H 7450 4150 50  0001 C CNN
+F 1 "+5V" H 7450 4440 50  0000 C CNN
+F 2 "" H 7450 4300 50  0000 C CNN
+F 3 "" H 7450 4300 50  0000 C CNN
+	1    7450 4300
 	1    0    0    -1
 $EndComp
@@
 L +24V #PWR?
 U 1 1 57D4AAF2
-P 6750 4550
-F 0 "#PWR?" H 6750 4400 50  0001 C CNN
-F 1 "+24V" H 6750 4690 50  0000 C CNN
-F 2 "" H 6750 4550 50  0000 C CNN
-F 3 "" H 6750 4550 50  0000 C CNN
-	1    6750 4550
-	1    0    0    -1
-$EndComp
-Wire Wire Line
-	6750 4550 6750 4700
-Wire Wire Line
-	6750 4700 6950 4700
+P 5400 4300
+F 0 "#PWR?" H 5400 4150 50  0001 C CNN
+F 1 "+24V" H 5400 4440 50  0000 C CNN
+F 2 "" H 5400 4300 50  0000 C CNN
+F 3 "" H 5400 4300 50  0000 C CNN
+	1    5400 4300
+	1    0    0    -1
+$EndComp
+Wire Wire Line
+	5400 4300 5400 4450
+Wire Wire Line
+	5400 4450 5600 4450
 $Comp
 L C C?
 U 1 1 57D4AE2C
-P 7450 5050
-F 0 "C?" H 7475 5150 50  0000 L CNN
-F 1 "100nF" H 7475 4950 50  0000 L CNN
-F 2 "Capacitors_SMD:C_0805_HandSoldering" V 7488 4900 50  0001 C CNN
-F 3 "" H 7450 5050 50  0000 C CNN
-	1    7450 5050
-	1    0    0    -1
-$EndComp
-Wire Wire Line
-	7450 4900 7450 4700
-Connection ~ 7450 4700
+P 6100 4800
+F 0 "C?" H 6125 4900 50  0000 L CNN
+F 1 "100nF" H 6125 4700 50  0000 L CNN
+F 2 "Capacitors_SMD:C_0805_HandSoldering" V 6138 4650 50  0001 C CNN
+F 3 "" H 6100 4800 50  0000 C CNN
+	1    6100 4800
+	1    0    0    -1
+$EndComp
+Wire Wire Line
+	6100 4650 6100 4450
+Connection ~ 6100 4450
 $Comp
 L GND #PWR?
 U 1 1 57D4B5C8
-P 7450 5250
-F 0 "#PWR?" H 7450 5000 50  0001 C CNN
-F 1 "GND" H 7450 5100 50  0000 C CNN
-F 2 "" H 7450 5250 50  0000 C CNN
-F 3 "" H 7450 5250 50  0000 C CNN
-	1    7450 5250
-	1    0    0    -1
-$EndComp
-Wire Wire Line
-	7450 5200 7450 5250
+P 6100 5000
+F 0 "#PWR?" H 6100 4750 50  0001 C CNN
+F 1 "GND" H 6100 4850 50  0000 C CNN
+F 2 "" H 6100 5000 50  0000 C CNN
+F 3 "" H 6100 5000 50  0000 C CNN
+	1    6100 5000
+	1    0    0    -1
+$EndComp
+Wire Wire Line
+	6100 4950 6100 5000
 $Comp
 L C C?
 U 1 1 57D4C8CC
-P 8800 5000
-F 0 "C?" H 8825 5100 50  0000 L CNN
-F 1 "10uF" H 8825 4900 50  0000 L CNN
-F 2 "Capacitors_SMD:C_0805_HandSoldering" V 8838 4850 50  0001 C CNN
-F 3 "" H 8800 5000 50  0000 C CNN
-	1    8800 5000
+P 7450 4750
+F 0 "C?" H 7475 4850 50  0000 L CNN
+F 1 "10uF" H 7475 4650 50  0000 L CNN
+F 2 "Capacitors_SMD:C_0805_HandSoldering" V 7488 4600 50  0001 C CNN
+F 3 "" H 7450 4750 50  0000 C CNN
+	1    7450 4750
 	1    0    0    -1
 $EndComp
@@
 L GND #PWR?
 U 1 1 57D4C95F
-P 8800 5250
-F 0 "#PWR?" H 8800 5000 50  0001 C CNN
-F 1 "GND" H 8800 5100 50  0000 C CNN
-F 2 "" H 8800 5250 50  0000 C CNN
-F 3 "" H 8800 5250 50  0000 C CNN
-	1    8800 5250
-	1    0    0    -1
-$EndComp
-Wire Wire Line
-	8800 4550 8800 4850
-Wire Wire Line
-	8400 4700 8800 4700
-Connection ~ 8800 4700
-Wire Wire Line
-	8800 5150 8800 5250
+P 7450 5000
+F 0 "#PWR?" H 7450 4750 50  0001 C CNN
+F 1 "GND" H 7450 4850 50  0000 C CNN
+F 2 "" H 7450 5000 50  0000 C CNN
+F 3 "" H 7450 5000 50  0000 C CNN
+	1    7450 5000
+	1    0    0    -1
+$EndComp
+Wire Wire Line
+	7450 4300 7450 4600
+Wire Wire Line
+	7050 4450 7450 4450
+Connection ~ 7450 4450
+Wire Wire Line
+	7450 4900 7450 5000
+$Comp
+L Q_PMOS_GSD Q?
+U 1 1 57DE64E8
+P 6700 1700
+F 0 "Q?" H 7000 1750 50  0000 R CNN
+F 1 "Q_PMOS_GSD" H 7350 1650 50  0000 R CNN
+F 2 "TO_SOT_Packages_THT:TO-220_Neutral123_Vertical" V 6900 1800 50  0001 C CNN
+F 3 "" H 6700 1700 50  0000 C CNN
+	1    6700 1700
+	1    0    0    -1
+$EndComp
+$Comp
+L FUSE F?
+U 1 1 57DE8225
+P 10500 2350
+F 0 "F?" H 10600 2400 50  0000 C CNN
+F 1 "FUSE" H 10400 2300 50  0000 C CNN
+F 2 "" H 10500 2350 50  0000 C CNN
+F 3 "" H 10500 2350 50  0000 C CNN
+	1    10500 2350
+	0    1    1    0
+$EndComp
+Wire Wire Line
+	10500 2600 10500 2650
+$Comp
+L R R?
+U 1 1 57DE8E45
+P 10400 1800
+F 0 "R?" V 10480 1800 50  0000 C CNN
+F 1 "R" V 10400 1800 50  0000 C CNN
+F 2 "" V 10330 1800 50  0000 C CNN
+F 3 "" H 10400 1800 50  0000 C CNN
+	1    10400 1800
+	1    0    0    -1
+$EndComp
+$Comp
+L R R?
+U 1 1 57DE8F01
+P 10600 1800
+F 0 "R?" V 10680 1800 50  0000 C CNN
+F 1 "R" V 10600 1800 50  0000 C CNN
+F 2 "" V 10530 1800 50  0000 C CNN
+F 3 "" H 10600 1800 50  0000 C CNN
+	1    10600 1800
+	1    0    0    -1
+$EndComp
+Wire Wire Line
+	10500 2100 10500 2000
+Wire Wire Line
+	10400 2000 10600 2000
+Wire Wire Line
+	10400 2000 10400 1950
+Wire Wire Line
+	10600 2000 10600 1950
+Connection ~ 10500 2000
+Wire Wire Line
+	10400 1650 10400 1550
+Wire Wire Line
+	10400 1550 10600 1550
+Wire Wire Line
+	10600 1550 10600 1650
+Connection ~ 10500 1550
+Wire Wire Line
+	10500 950  10500 1550
+Wire Wire Line
+	10050 1250 10500 1250
+Connection ~ 10500 1250
+Text Label 10100 1250 0    60   ~ 0
+v_i
+$Comp
+L LM358 U?
+U 1 1 57DEBEED
+P 9100 4900
+F 0 "U?" H 9050 5100 50  0000 L CNN
+F 1 "LM358" H 9050 4650 50  0000 L CNN
+F 2 "" H 9100 4900 50  0000 C CNN
+F 3 "" H 9100 4900 50  0000 C CNN
+	1    9100 4900
+	-1   0    0    1
+$EndComp
 $EndSCHEMATC
