File: current-source-stm8/current-source-stm8.sch (KiCad schematic (older format))
At the start: 38 parts

Commit message: add pcb current-source
Parts:
- removed Q?: Q_NMOS_DGS, symbol Q_NMOS_DGS
- removed U?: LM358, symbol LM358
- removed U?: LM7805, symbol LM7805
- added C6, C8: 100nF, Capacitors_SMD:C_0805_HandSoldering, symbol C
- added Q2: Q_PMOS_GSD, TO_SOT_Packages_THT:TO-220_Neutral123_Vertical, symbol Q_PMOS_GSD
- added R10: R, Resistors_ThroughHole:Resistor_Horizontal_RM10mm, symbol R
- added R7: 0.15, Resistors_ThroughHole:Resistor_Horizontal_RM20mm, symbol R
- added U1: LM7805CT, TO_SOT_Packages_SMD:TO-252-2Lead, symbol LM7805CT
- added U2: LM358, symbol LM358
- C1, C7: renamed from C?; footprint (none) -> Capacitors_SMD:C_1206_HandSoldering
- C10: renamed from C?; value C -> 1uF; footprint (none) -> Capacitors_SMD:C_0805_HandSoldering
- C11, C3, C4, C9: renamed from C?; footprint (none) -> Capacitors_SMD:C_0805_HandSoldering
- C2, C5: renamed from C?; footprint (none) -> Capacitors_SMD:c_elec_8x10
- D1, D3: renamed from D?; footprint (none) -> Diodes_SMD:SOD-123
- D2, D4: renamed from D?; footprint (none) -> Diodes_SMD:DO-214AB_Handsoldering
- D5: renamed from D?; footprint (none) -> LEDs:LED_0805
- F1: renamed from F?; footprint (none) -> Fuse_Holders_and_Fuses:Fuse_SMD2920
- IC1: renamed from IC?; footprint TSSOP-20 -> Housings_SSOP:TSSOP-20_4.4x6.5mm_Pitch0.65mm
- L1: renamed from L?; footprint (none) -> Inductors:SELF-WE-PD-XXL
- P1, P2: renamed from P?; footprint (none) -> Terminal_Blocks:TerminalBlock_Pheonix_PT-3.5mm_2pol
- P3: renamed from P?; footprint (none) -> Pin_Headers:Pin_Header_Straight_1x04
- Q1, Q4: renamed from Q?; footprint TO-220 -> TO_SOT_Packages_SMD:SOT-23
- Q3: renamed from Q?; footprint (none) -> TO_SOT_Packages_SMD:SOT-23
- R1, R11, R12, R13, R14, R2, R3, R4, R5, R8: renamed from R?; footprint (none) -> Resistors_SMD:R_0805_HandSoldering
- R6: renamed from 0.15; value R -> 0.15; footprint (none) -> Resistors_ThroughHole:Resistor_Horizontal_RM20mm
- R9: renamed from R?; footprint (none) -> Resistors_ThroughHole:Resistor_Horizontal_RM10mm
Connections:
- wire segments 87 -> 97
